Commit message: fix collision

File: smartbots/assets/Manipulators/braccio.urdf (robot description, URDF)
Before this commit: robot braccio, 9 links, 8 joints
Links:
- link base_link: geometry collision box size=0.15 0.15 .05; visual box size=0.15 0.15 .05
- link gripper_base: geometry collision mesh filename=package://Smartbots/smartbots/assets/meshes/braccio/gripper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; visual mesh filename=package://Smartbots/smartbots/assets/meshes/braccio/gripper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
- link gripper_fix: geometry collision mesh filename=package://Smartbots/smartbots/assets/meshes/braccio/gripper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; visual mesh filename=package://Smartbots/smartbots/assets/meshes/braccio/gripper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
- link gripper_movable: geometry collision mesh filename=package://Smartbots/smartbots/assets/meshes/braccio/gripper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; visual mesh filename=package://Smartbots/smartbots/assets/meshes/braccio/gripper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
- link link1: geometry collision mesh filename=package://Smartbots/smartbots/assets/meshes/braccio/base.stl; visual mesh filename=package://Smartbots/smartbots/assets/meshes/braccio/base.stl
- link link2: geometry collision mesh filename=package://Smartbots/smartbots/assets/meshes/braccio/shoulde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; visual mesh filename=package://Smartbots/smartbots/assets/meshes/braccio/shoulde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
- link link3: geometry collision mesh filename=package://Smartbots/smartbots/assets/meshes/braccio/elbow.s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; visual mesh filename=package://Smartbots/smartbots/assets/meshes/braccio/elbow.s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
- link link4: geometry collision mesh filename=package://Smartbots/smartbots/assets/meshes/braccio/wrist_p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; visual mesh filename=package://Smartbots/smartbots/assets/meshes/braccio/wrist_p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
- link link5: geometry collision mesh filename=package://Smartbots/smartbots/assets/meshes/braccio/wrist_r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; visual mesh filename=package://Smartbots/smartbots/assets/meshes/braccio/wrist_r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
